File: battery-protector-v2.sch (KiCad schematic (older format))
At the start: 28 parts, among them J1 Conn_01x04, J2 Anderson_two_redblack, J3 Anderson_two_redblack, P1 10118194, SW1 SW_SPST, SW2 OS102011MS2QN1, U1 SAMD21E18, U2 WS2812b, U3 MIC5203, U4 MOSFET_CSD17318Q2

Commit message: Board v1.0
Parts:
- removed RV1: POT, homebrew:BOURNS_PDB12H_POT, symbol POT
Connections:
- net labels removed: KNOB
- no-connect marks 19 -> 20
Changed lines of the file:
@@
 Wire Wire Line
 	5650 4950 5650 5000
-Text GLabel 2250 1550 2    60   Input ~ 0
-KNOB
-$Comp
-L POT RV1
-U 1 1 5B5181A4
-P 6550 4850
-F 0 "RV1" V 6375 4850 50  0000 C CNN
-F 1 "POT" V 6450 4850 50  0000 C CNN
-F 2 "homebrew:BOURNS_PDB12H_POT" H 6550 4850 50  0001 C CNN
-F 3 "" H 6550 4850 50  0001 C CNN
-	1    6550 4850
-	1    0    0    -1
-$EndComp
-$Comp
-L VCC #PWR026
-U 1 1 5B518324
-P 6550 4700
-F 0 "#PWR026" H 6550 4550 50  0001 C CNN
-F 1 "VCC" H 6550 4850 50  0000 C CNN
-F 2 "" H 6550 4700 50  0001 C CNN
-F 3 "" H 6550 4700 50  0001 C CNN
-	1    6550 4700
-	1    0    0    -1
-$EndComp
-$Comp
-L GND #PWR027
-U 1 1 5B51837A
-P 6550 5000
-F 0 "#PWR027" H 6550 4750 50  0001 C CNN
-F 1 "GND" H 6550 4850 50  0000 C CNN
-F 2 "" H 6550 5000 50  0001 C CNN
-F 3 "" H 6550 5000 50  0001 C CNN
-	1    6550 5000
-	1    0    0    -1
-$EndComp
-Text GLabel 6700 4850 2    60   Input ~ 0
-KNOB
 NoConn ~ 2250 1050
 NoConn ~ 2250 1150
@@
 	1    0    0    -1
 $EndComp
+NoConn ~ 2250 1550
 $EndSCHEMATC
